File: io.kicad_sch (KiCad schematic)
At the start: 28 parts, among them SW10 RotaryEncoder, SW11 RotaryEncoder, SW12 RotaryEncoder, SW13 RotaryEncoder, SW14 RotaryEncoder, SW7 RotaryEncoder, SW8 RotaryEncoder, SW9 RotaryEncoder, U1 MCP23017_SO

Commit message: Add bom
Parts:
- SW10, SW11, SW12, SW13, SW14, SW7, SW8, SW9: Comment (none) -> without switch
Changed lines of the file:
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@@
+      (effects (font (size 1.27 1.27)) hide)
+    )
+    (property "Comment" "" (at 135.89 39.37 0)
       (effects (font (size 1.27 1.27)) hide)
     )
@@
     )
     (property "Datasheet" "~" (at 53.34 139.7 0)
+      (effects (font (size 1.27 1.27)) hide)
+    )
+    (property "Comment" "" (at 53.34 139.7 0)
       (effects (font (size 1.27 1.27)) hide)
     )
@@
       (effects (font (size 1.27 1.27)) hide)
     )
+    (property "Comment" "" (at 55.88 91.44 0)
+      (effects (font (size 1.27 1.27)) hide)
+    )
     (pin "1")
     (pin "2")
@@
     )
     (property "Datasheet" "~" (at 213.36 59.436 0)
+      (effects (font (size 1.27 1.27)) hide)
+    )
+    (property "Comment" "without switch" (at 213.36 66.04 0)
       (effects (font (size 1.27 1.27)) hide)
     )
@@
       (effects (font (size 1.27 1.27)) hide)
     )
+    (property "Comment" "" (at 147.32 39.37 0)
+      (effects (font (size 1.27 1.27)) hide)
+    )
     (pin "1")
     (pin "2")
@@
       (effects (font (size 1.27 1.27)) hide)
     )
+    (property "Comment" "" (at 185.42 39.37 0)
+      (effects (font (size 1.27 1.27)) hide)
+    )
     (pin "1")
     (pin "2")
@@
     )
     (property "Datasheet" "~" (at 173.99 39.37 0)
+      (effects (font (size 1.27 1.27)) hide)
+    )
+    (property "Comment" "" (at 173.99 39.37 0)
       (effects (font (size 1.27 1.27)) hide)
     )
@@
       (effects (font (size 1.27 1.27)) hide)
     )
+    (property "Comment" "" (at 158.75 39.37 0)
+      (effects (font (size 1.27 1.27)) hide)
+    )
     (pin "1")
     (pin "2")
@@
     (property "Datasheet" "http://ww1.microchip.com/downloads/en/DeviceDoc/20001952C.pdf" (at 93.98 121.92 0)
       (effects (font (size 1.27 1.27)) (justify left) hide)
+    )
+    (property "Comment" "" (at 88.9 93.98 0)
+      (effects (font (size 1.27 1.27)) hide)
     )
     (pin "1")
@@
       (effects (font (size 1.27 1.27)) hide)
     )
+    (property "Comment" "" (at 132.08 39.37 0)
+      (effects (font (size 1.27 1.27)) hide)
+    )
     (pin "1")
     (pin "2")
@@
     )
     (property "Datasheet" "~" (at 213.36 48.006 0)
+      (effects (font (size 1.27 1.27)) hide)
+    )
+    (property "Comment" "without switch" (at 213.36 54.61 0)
       (effects (font (size 1.27 1.27)) hide)
     )
@@
       (effects (font (size 1.27 1.27)) hide)
     )
+    (property "Comment" "" (at 170.18 39.37 0)
+      (effects (font (size 1.27 1.27)) hide)
+    )
     (pin "1")
     (pin "2")
@@
       (effects (font (size 1.27 1.27)) hide)
     )
+    (property "Comment" "" (at 189.23 39.37 0)
+      (effects (font (size 1.27 1.27)) hide)
+    )
     (pin "1")
     (pin "2")
@@
       (effects (font (size 1.27 1.27)) hide)
     )
+    (property "Comment" "" (at 177.8 39.37 0)
+      (effects (font (size 1.27 1.27)) hide)
+    )
     (pin "1")
     (pin "2")
@@
       (effects (font (size 1.27 1.27)) hide)
     )
+    (property "Comment" "" (at 139.7 39.37 0)
+      (effects (font (size 1.27 1.27)) hide)
+    )
     (pin "1")
     (pin "2")
@@
     )
     (property "Datasheet" "~" (at 213.36 128.016 0)
+      (effects (font (size 1.27 1.27)) hide)
+    )
+    (property "Comment" "without switch" (at 213.36 134.62 0)
       (effects (font (size 1.27 1.27)) hide)
     )
@@
       (effects (font (size 1.27 1.27)) hide)
     )
+    (property "Comment" "" (at 55.88 88.9 0)
+      (effects (font (size 1.27 1.27)) hide)
+    )
     (pin "1")
     (pin "2")
@@
       (effects (font (size 1.27 1.27)) hide)
     )
+    (property "Comment" "" (at 154.94 39.37 0)
+      (effects (font (size 1.27 1.27)) hide)
+    )
     (pin "1")
     (pin "2")
@@
     )
     (property "Datasheet" "~" (at 213.36 70.866 0)
+      (effects (font (size 1.27 1.27)) hide)
+    )
+    (property "Comment" "without switch" (at 213.36 77.47 0)
       (effects (font (size 1.27 1.27)) hide)
     )
@@
       (effects (font (size 1.27 1.27)) hide)
     )
+    (property "Comment" "without switch" (at 213.36 111.76 0)
+      (effects (font (size 1.27 1.27)) hide)
+    )
     (pin "A")
     (pin "B")
@@
       (effects (font (size 1.27 1.27)) hide)
     )
+    (property "Comment" "without switch" (at 213.36 100.33 0)
+      (effects (font (size 1.27 1.27)) hide)
+    )
     (pin "A")
     (pin "B")
@@
       (effects (font (size 1.27 1.27)) hide)
     )
+    (property "Comment" "" (at 151.13 39.37 0)
+      (effects (font (size 1.27 1.27)) hide)
+    )
     (pin "1")
     (pin "2")
@@
     )
     (property "Datasheet" "~" (at 181.61 39.37 0)
+      (effects (font (size 1.27 1.27)) hide)
+    )
+    (property "Comment" "" (at 181.61 39.37 0)
       (effects (font (size 1.27 1.27)) hide)
     )
@@
       (effects (font (size 1.27 1.27)) hide)
     )
+    (property "Comment" "" (at 166.37 39.37 0)
+      (effects (font (size 1.27 1.27)) hide)
+    )
     (pin "1")
     (pin "2")
@@
       (effects (font (size 1.27 1.27)) hide)
     )
+    (property "Comment" "" (at 143.51 39.37 0)
+      (effects (font (size 1.27 1.27)) hide)
+    )
     (pin "1")
     (pin "2")
@@
     )
     (property "Datasheet" "~" (at 213.36 116.586 0)
+      (effects (font (size 1.27 1.27)) hide)
+    )
+    (property "Comment" "without switch" (at 213.36 123.19 0)
       (effects (font (size 1.27 1.27)) hide)
     )
@@
       (effects (font (size 1.27 1.27)) hide)
     )
+    (property "Comment" "without switch" (at 213.36 88.9 0)
+      (effects (font (size 1.27 1.27)) hide)
+    )
     (pin "A")
     (pin "B")
@@
       (effects (font (size 1.27 1.27)) hide)
     )
+    (property "Comment" "" (at 162.56 39.37 0)
+      (effects (font (size 1.27 1.27)) hide)
+    )
