File: polykit-x-controlboard.kicad_sch (KiCad schematic)
At the start: 12 parts, among them J1 MCU_BOARD, J2 X8_I2C_POWER, J3 X8_EXT_DIGITAL, J4 DISPLAY, SW1 SW_Push, SW2 SW_Push, SW3 SW_Push, SW4 SW_Push, SW5 SW_Push, SW6 SW_Push

Commit message: Add bom
Parts:
- J1: Comment (none) -> optional, when used as MIDI controller
Changed lines of the file:
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@@
+      (effects (font (size 1.27 1.27)) hide)
+    )
+    (property "Comment" "" (at 238.76 35.56 0)
       (effects (font (size 1.27 1.27)) hide)
     )
@@
       (effects (font (size 1.27 1.27)) hide)
     )
+    (property "Comment" "" (at 191.77 138.43 0)
+      (effects (font (size 1.27 1.27)) hide)
+    )
     (pin "1")
     (pin "2")
@@
       (effects (font (size 1.27 1.27)) hide)
     )
+    (property "Comment" "" (at 162.56 50.8 0)
+      (effects (font (size 1.27 1.27)) hide)
+    )
     (pin "1")
     (pin "2")
@@
     )
     (property "Datasheet" "~" (at 162.56 86.36 0)
+      (effects (font (size 1.27 1.27)) hide)
+    )
+    (property "Comment" "" (at 162.56 91.44 0)
       (effects (font (size 1.27 1.27)) hide)
     )
@@
     )
     (property "Datasheet" "~" (at 227.33 54.61 0)
+      (effects (font (size 1.27 1.27)) hide)
+    )
+    (property "Comment" "" (at 227.33 54.61 0)
       (effects (font (size 1.27 1.27)) hide)
     )
@@
       (effects (font (size 1.27 1.27)) hide)
     )
+    (property "Comment" "" (at 162.56 40.64 0)
+      (effects (font (size 1.27 1.27)) hide)
+    )
     (pin "1")
     (pin "2")
@@
     )
     (property "Datasheet" "~" (at 227.33 85.09 0)
+      (effects (font (size 1.27 1.27)) hide)
+    )
+    (property "Comment" "" (at 227.33 85.09 0)
       (effects (font (size 1.27 1.27)) hide)
     )
@@
       (effects (font (size 1.27 1.27)) hide)
     )
+    (property "Comment" "optional, when used as MIDI controller" (at 137.16 144.78 0)
+      (effects (font (size 1.27 1.27)) hide)
+    )
     (pin "1")
     (pin "10")
@@
       (effects (font (size 1.27 1.27)) hide)
     )
+    (property "Comment" "" (at 219.71 35.56 0)
+      (effects (font (size 1.27 1.27)) hide)
+    )
     (pin "1")
     (pin "2")
@@
       (effects (font (size 1.27 1.27)) hide)
     )
+    (property "Comment" "" (at 162.56 60.96 0)
+      (effects (font (size 1.27 1.27)) hide)
+    )
     (pin "1")
     (pin "2")
@@
       (effects (font (size 1.27 1.27)) hide)
     )
+    (property "Comment" "" (at 162.56 81.28 0)
+      (effects (font (size 1.27 1.27)) hide)
+    )
     (pin "1")
     (pin "2")
@@
       (effects (font (size 1.27 1.27)) hide)
     )
+    (property "Comment" "" (at 162.56 71.12 0)
+      (effects (font (size 1.27 1.27)) hide)
+    )
